File: hardware/mixer/mixer.kicad_pcb (KiCad board)
At the start: 2 copper layers, 40 x 100 mm, 63 parts, among them J1 AudioJack2_SwitchT, J2 AudioJack2_SwitchT, J3 AudioJack2_SwitchT, J5 AudioJack2_SwitchT, J6 AudioJack2_SwitchT, J7 AudioJack2_SwitchT, J8 AudioJack2_SwitchT, J9 Conn_02x08_Odd_Even, Q5 2N3906, Q6 2N3904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

Commit message: changed R15 to 68k
Parts:
- R15: value 47k -> 68k
Changed lines of the file:
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@@
 			)
 		)
-		(property "Value" "47k"
+		(property "Value" "68k"
 			(at 1.27 1.92 0)
 			(layer "F.Fab")
